Commit message: Fix wheel links and wheel joints numbers.

File: robotino_description/robotino.urdf (robot description, URDF)
Before this commit: robot robotino, 4 links, 3 joints
Links:
- added link platform_link; collision mesh filename=package://robotino_description/model/Robotino3_Platform.dae scale=0.009 0.009 0.009; visual mesh filename=package://robotino_description/model/Robotino3_Platform.dae scale=0.009 0.009 0.009
Joints:
- added joint platform_joint: type fixed, parent base_link, child platform_link, origin xyz=0 0 0 rpy=0 0 0, axis 0 0 0
- joint wheel0_joint: origin xyz=-0.0001 0.1825 0.059154 rpy=0 0 0 -> xyz=0.156867 -0.090625 0.059154 rpy=0 0 -2.094395102393195
- joint wheel1_joint: origin xyz=-0.157067 -0.090625 0.059154 rpy=0 0 2.094395102393195 -> xyz=-0.0001 0.1825 0.059154 rpy=0 0 0
- joint wheel2_joint: origin xyz=0.156867 -0.090625 0.059154 rpy=0 0 -2.094395102393195 -> xyz=-0.157067 -0.090625 0.059154 rpy=0 0 2.094395102393195
