Commit message: Fix orientation of platform in robotino.urdf.xacro.

File: robotino_description/robotino.urdf.xacro (robot description, xacro)
@@ -74,6 +74,5 @@
     <parent link="base_link"/>
     <child link="platform_link"/>
-    <origin xyz="0 0 0" rpy="0 0 0"/>
-    <axis xyz="0 0 0" rpy="0 0 0"/>
+    <origin xyz="0 0 0" rpy="0 0 ${PI/2}"/>
   </joint>
 </robot>

Commit message: Add mesh of laser range finder Hokuyo URG-04LX-UG01. Add laser range finder in robotino.urdf.xacro.

File: robotino_description/robotino.urdf.xacro (robot description, xacro)
@@ -58,4 +58,28 @@
   <xacro:range_sensor name="ir7" angle="${7*sensor_delta_angle}"/>
   <xacro:range_sensor name="ir8" angle="${8*sensor_delta_angle}"/>
+  <xacro:macro name="laser_range_finder" params="parent *origin">
+    <link name="laser_base">
+      <visual>
+        <origin xyz="0 0 0" rpy="0 0 0"/>
+        <geometry>
+          <mesh filename="package://robotino_description/model/hokuyo.dae" scale="1 1 1"/>
+        </geometry>
+      </visual>
+    </link>
+    <link name="laser_link"></link>
+    <joint name="laser_link_joint" type="fixed">
+      <parent link="laser_base"/>
+      <child link="laser_link"/>
+      <origin xyz="0 0 0.05775" rpy="0 0 0"/>
+    </joint>
+    <joint name="laser_joint" type="fixed">
+      <parent link="${parent}"/>
+      <child link="laser_base"/>
+      <xacro:insert_block name="origin"/>
+    </joint>
+  </xacro:macro>
+  <xacro:laser_range_finder parent="base_link">
+    <origin xyz="0.091 0 0.1915" rpy="0 0 0"/>
+  </xacro:laser_range_finder>
   <link name="platform_link">
     <visual>

Commit message: Rename model directory to meshes in robotino_description package.

File: robotino_description/robotino.urdf.xacro (robot description, xacro)
@@ -7,5 +7,5 @@
       <origin xyz="0 0 0.035" rpy="0 0 ${PI/2}"/>
       <geometry>
-        <mesh filename="package://robotino_description/model/Robotino3_SplitMain.dae" scale="0.01 0.01 0.01"/>
+        <mesh filename="package://robotino_description/meshes/Robotino3_SplitMain.dae" scale="0.01 0.01 0.01"/>
       </geometry>
     </visual>
@@ -24,5 +24,5 @@
         <origin xyz="0 0 0" rpy="0 0 0"/>
         <geometry>
-          <mesh filename="package://robotino_description/model/Robotino3_SplitWheel.dae" scale="0.01 0.01 0.01"/>
+          <mesh filename="package://robotino_description/meshes/Robotino3_SplitWheel.dae" scale="0.01 0.01 0.01"/>
         </geometry>
       </visual>
@@ -63,5 +63,5 @@
         <origin xyz="0 0 0" rpy="0 0 0"/>
         <geometry>
-          <mesh filename="package://robotino_description/model/hokuyo.dae" scale="1 1 1"/>
+          <mesh filename="package://robotino_description/meshes/hokuyo.dae" scale="1 1 1"/>
         </geometry>
       </visual>
@@ -86,10 +86,10 @@
       <origin xyz="0 0 0" rpy="0 0 0"/>
       <geometry>
-        <mesh filename="package://robotino_description/model/Robotino3_Platform.dae" scale="0.009 0.009 0.009"/>
+        <mesh filename="package://robotino_description/meshes/Robotino3_Platform.dae" scale="0.009 0.009 0.009"/>
       </geometry>
     </visual>
     <collision>
       <geometry>
-        <mesh filename="package://robotino_description/model/Robotino3_Platform.dae" scale="0.009 0.009 0.009"/>
+        <mesh filename="package://robotino_description/meshes/Robotino3_Platform.dae" scale="0.009 0.009 0.009"/>
       </geometry>
     </collision>
