Commit message: Fix collisions.

File: robotino_description/urdf/_tower_with_segments.urdf.xacro (robot description, xacro)
@@ -1,4 +1,7 @@
 <?xml version="1.0"?>
 <robot xmlns:xacro="http://www.ros.org/wiki/xacro" name="tower_with_segments">
+  <xacro:property name="segment_radius" value="0.225"/>
+  <xacro:property name="tower_height" value="0.5775"/>
+  <xacro:property name="tower_shift" value="0.1915"/>
   <link name="tower_link">
     <visual>
@@ -9,6 +12,7 @@
     </visual>
     <collision>
+      <origin xyz="0 0 ${tower_height/2 + tower_shift}" rpy="0 0 0"/>
       <geometry>
-        <mesh filename="package://robotino_description/meshes/TowerWithSegments.dae" scale="0.01 0.01 0.01"/>
+        <cylinder length="${tower_height}" radius="${segment_radius}"/>
       </geometry>
     </collision>

File: robotino_description/urdf/robotino3.urdf.xacro (robot description, xacro)
@@ -4,4 +4,5 @@
   <xacro:property name="base_height" value="0.325"/>
   <xacro:property name="base_mass" value="21.4"/> <!-- with 2 accumulators -->
+  <xacro:property name="base_clearance" value="0.019"/>
   <link name="base_link">
     <visual>
@@ -12,5 +13,5 @@
     </visual>
     <collision>
-      <origin xyz="0 0 ${base_height/2}" rpy="0 0 0"/>
+      <origin xyz="0 0 ${base_height/2 + base_clearance}" rpy="0 0 0"/>
       <geometry>
         <cylinder length="${base_height}" radius="${base_radius}"/>
@@ -18,5 +19,5 @@
     </collision>
     <inertial>
-      <origin xyz="0 0 ${base_height/2}" rpy="0 0 ${radians(90)}"/>
+      <origin xyz="0 0 ${base_height/2 + base_clearance}" rpy="0 0 ${radians(90)}"/>
       <mass value="${base_mass}"/>
       <inertia ixx="${base_mass*(3*base_radius**2 + base_height**2)/12}" ixy="0.0" ixz="0.0"

File: robotino_description/urdf/robotino4.urdf.xacro (robot description, xacro)
@@ -4,4 +4,5 @@
   <xacro:property name="base_height" value="0.325"/>
   <xacro:property name="base_mass" value="21.4"/> <!-- with 2 accumulators -->
+  <xacro:property name="base_clearance" value="0.019"/>
   <link name="base_link">
     <visual>
@@ -12,5 +13,5 @@
     </visual>
     <collision>
-      <origin xyz="0 0 ${base_height/2}" rpy="0 0 0"/>
+      <origin xyz="0 0 ${base_height/2 + base_clearance}" rpy="0 0 0"/>
       <geometry>
         <cylinder length="${base_height}" radius="${base_radius}"/>
@@ -18,5 +19,5 @@
     </collision>
     <inertial>
-      <origin xyz="0 0 ${base_height/2}" rpy="0 0 ${radians(90)}"/>
+      <origin xyz="0 0 ${base_height/2 + base_clearance}" rpy="0 0 ${radians(90)}"/>
       <mass value="${base_mass}"/>
       <inertia ixx="${base_mass*(3*base_radius**2 + base_height**2)/12}" ixy="0.0" ixz="0.0"
