Commit message: Add collision of hokuyo laser range finder.

File: robotino_description/urdf/sensors/hokuyo_laser_range_finder.urdf.xacro (robot description, xacro)
@@ -2,4 +2,6 @@
 <robot xmlns:xacro="http://www.ros.org/wiki/xacro">
   <xacro:macro name="laser_range_finder" params="parent *origin">
+    <xacro:property name="laser_height" value="0.07"/>
+    <xacro:property name="laser_size" value="0.05"/>
     <link name="laser_base">
       <visual>
@@ -9,4 +11,10 @@
         </geometry>
       </visual>
+      <collision>
+        <origin xyz="0 0 ${laser_height/2}" rpy="0 ${radians(90)} 0"/>
+        <geometry>
+          <box size="${laser_height} ${laser_size} ${laser_size}"/>
+        </geometry>
+      </collision>
     </link>
     <link name="laser_link"></link>
