Commit message: Finish integration of robotino_camera_node.
Fix CameraROS: associate the camera with the Com object and process Com events,
stamp camera_info, skip undecoded and truncated images. Load camera calibration
with camera_info_manager (camera_info_url parameter, /set_camera_info service).
Add frame_id, image resolution and format parameters.

Add camera_optical_frame to Logitech C920 URDF, launch the camera node from
rto_bringup_launch.py, show the image in RViz, document the camera node in README.

Co-Authored-By: Claude Opus 5.5 <noreply@anthropic.com>

File: robotino_description/urdf/sensors/logitech_c920.urdf.xacro (robot description, xacro)
@@ -8,4 +8,11 @@
         <xacro:insert_block name="origin"/>
     </joint>
+    <!-- Frame of camera images: z forward, x right, y down -->
+    <link name="camera_optical_frame"></link>
+    <joint name="camera_optical_joint" type="fixed">
+        <parent link="camera_link"/>
+        <child link="camera_optical_frame"/>
+        <origin xyz="0 0 0" rpy="${-pi/2} 0 ${-pi/2}"/>
+    </joint>
   </xacro:macro>
 </robot>
