Commit message: Add gazebo_sim.launch.py. Replace meshes filenames from "package://package_name" to "$(find <package_name>)", because gazebo requires absolute path to meshes. Replace running of xacro in installation time to running of xacro in launch time.

File: robotino_description/urdf/robotino3/omniwheel.urdf.xacro (robot description, xacro)
@@ -10,5 +10,5 @@
         <origin xyz="0 0 0" rpy="0 0 0"/>
         <geometry>
-          <mesh filename="package://robotino_description/meshes/robotino3/omniwheel_rotacaster_r3_1258_85.dae" scale="0.01 0.01 0.01"/>
+          <mesh filename="file://$(find robotino_description)/meshes/robotino3/omniwheel_rotacaster_r3_1258_85.dae" scale="0.01 0.01 0.01"/>
         </geometry>
       </visual>

File: robotino_description/urdf/robotino4/omniwheel.urdf.xacro (robot description, xacro)
@@ -10,5 +10,5 @@
         <origin xyz="0 0 0" rpy="0 0 0"/>
         <geometry>
-          <mesh filename="package://robotino_description/meshes/robotino4/omniwheel_rotacaster_r2_1258_85.dae" scale="1 1 1"/>
+          <mesh filename="file://$(find robotino_description)/meshes/robotino4/omniwheel_rotacaster_r2_1258_85.dae" scale="1 1 1"/>
         </geometry>
       </visual>
