Commit message: Invert wheel joint direction to match ros2_control omni_wheel_drive_controller.
Positive wheel joint rotation now drives the robot clockwise around its center, as omni_wheel_drive_controller expects. robotino_node inverts the Robotino API2 motor readings accordingly, so /joint_states of the real robot stay consistent with the URDF.

Co-Authored-By: Claude Opus 5.5 <noreply@anthropic.com>

File: robotino_description/urdf/robotino3/omniwheel.urdf.xacro (robot description, xacro)
@@ -30,5 +30,5 @@
       <child link="${name}_link"/>
       <origin xyz="${wheel_distance * cos(angle)} ${wheel_distance * sin(angle)} ${wheel_radius}" rpy="0 0 ${angle + radians(90)}"/>
-      <axis xyz="0 1 0" rpy="0 0 0"/>
+      <axis xyz="0 -1 0" rpy="0 0 0"/>
     </joint>
   </xacro:macro>

File: robotino_description/urdf/robotino4/omniwheel.urdf.xacro (robot description, xacro)
@@ -30,5 +30,5 @@
       <child link="${name}_link"/>
       <origin xyz="${wheel_distance * cos(angle)} ${wheel_distance * sin(angle)} ${wheel_radius}" rpy="0 0 ${angle}"/>
-      <axis xyz="-1 0 0" rpy="0 0 0"/>
+      <axis xyz="1 0 0" rpy="0 0 0"/>
     </joint>
   </xacro:macro>

Commit message: Use a thin disk as omniwheel collision.
Physics engines put cylinder contacts on its rims, so the 43 mm wide wheel cylinder rolled on its inner edge in Gazebo and the robot rotated 12.5% faster than wheel odometry. A 4 mm disk keeps the ground contact near the wheel mid-plane.

Co-Authored-By: Claude Opus 5.5 <noreply@anthropic.com>

File: robotino_description/urdf/robotino3/omniwheel.urdf.xacro (robot description, xacro)
@@ -4,4 +4,5 @@
     <xacro:property name="wheel_radius" value="0.0625"/>
     <xacro:property name="wheel_thickness" value="0.062"/>
+    <xacro:property name="wheel_collision_thickness" value="0.004"/>
     <xacro:property name="wheel_mass" value="0.485"/>
     <xacro:property name="wheel_distance" value="0.1811"/>
@@ -13,8 +14,10 @@
         </geometry>
       </visual>
+      <!-- Physics engines put cylinder contacts on its rims, so a thin disk is used to keep
+           the ground contact close to the wheel mid-plane, like the rollers of a real omniwheel -->
       <collision>
         <origin xyz="0 0 0" rpy="${radians(90)} 0 0"/>
         <geometry>
-          <cylinder length="${wheel_thickness}" radius="${wheel_radius}"/>
+          <cylinder length="${wheel_collision_thickness}" radius="${wheel_radius}"/>
         </geometry>
       </collision>

File: robotino_description/urdf/robotino4/omniwheel.urdf.xacro (robot description, xacro)
@@ -4,4 +4,5 @@
     <xacro:property name="wheel_radius" value="0.0625"/>
     <xacro:property name="wheel_thickness" value="0.043"/>
+    <xacro:property name="wheel_collision_thickness" value="0.004"/>
     <xacro:property name="wheel_mass" value="0.315"/>
     <xacro:property name="wheel_distance" value="0.1911"/>
@@ -13,8 +14,10 @@
         </geometry>
       </visual>
+      <!-- Physics engines put cylinder contacts on its rims, so a thin disk is used to keep
+           the ground contact close to the wheel mid-plane, like the rollers of a real omniwheel -->
       <collision>
         <origin xyz="0 0 0" rpy="0 ${radians(90)} 0"/>
         <geometry>
-          <cylinder length="${wheel_thickness}" radius="${wheel_radius}"/>
+          <cylinder length="${wheel_collision_thickness}" radius="${wheel_radius}"/>
         </geometry>
       </collision>
