Commit message: Match simulated laser scan to Hokuyo URG-04LX-UG01 specification.
Use the sensor's measuring steps 44..725 of 1024 per revolution with step 384 straight ahead (-119.53..+119.88 deg, 682 points) and the 20 mm minimum range, as given by the SCIP 2.0 protocol specification (C-42-03320B).

Co-Authored-By: Claude Opus 5.5 <noreply@anthropic.com>

File: robotino_gazebo/urdf/robotino_sensors.urdf.xacro (robot description, xacro)
@@ -10,6 +10,10 @@
        Raw gz topics live under robotino/sim/ and are converted to robotino_node
        compatible ROS topics by ros_gz_bridge and sim_adapter.py. -->
-  <!-- Hokuyo URG-04LX: 240 deg, 683 steps, up to 5.6 m -->
+  <!-- Hokuyo URG-04LX-UG01: 240 deg field of view, 1024 steps per revolution (0.352 deg),
+       measuring steps 44..725 with step 384 straight ahead, 20..5600 mm, 100 ms per scan
+       (URG Series Communication Protocol Specification SCIP 2.0, C-42-03320B, PP command).
+       Accuracy is +-30 mm up to 1 m and +-3 % beyond, approximated by constant noise. -->
   <xacro:macro name="laser_range_finder_sim" params="frame:=laser_link">
+    <xacro:property name="laser_step" value="${2*pi/1024}"/>
     <gazebo reference="${frame}">
       <sensor name="laser" type="gpu_lidar">
@@ -21,12 +25,12 @@
           <scan>
             <horizontal>
-              <samples>683</samples>
+              <samples>${725 - 44 + 1}</samples>
               <resolution>1</resolution>
-              <min_angle>${radians(-120)}</min_angle>
-              <max_angle>${radians(120)}</max_angle>
+              <min_angle>${(44 - 384) * laser_step}</min_angle>
+              <max_angle>${(725 - 384) * laser_step}</max_angle>
             </horizontal>
           </scan>
           <range>
-            <min>0.06</min>
+            <min>0.02</min>
             <max>5.6</max>
             <resolution>0.001</resolution>
